File: ROFLtemp_1.kicad_pcb (KiCad board)
At the start: 2 copper layers, 141 parts, among them J1 USB_OTG, J2 CONN_02X05, P1 CONN_01X02, P2 CONN_01X02, P3 CONN_01X02, P4 CONN_01X02, Q1 ASEM1, Q10 DMN1019USN, Q11 DMP1100UCB4, Q12 DMN1019USN, Q2 DMN1019USN, Q3 DMN1019USN, Q4 DMP1100UCB4, Q5 DMN1019USN, Q6 DMN1019USN, Q7 DMP1100UCB4, Q8 DMN1019USN, Q9 DMN1019USN, SW1 SW_SPST, U1 TPS2290x, U2 BQ24079, U3 MAX31865, U4 STM32F042K6Tx, U5 TPS63051, U6 7SEGMENT_CA, U7 7SEGMENT_CA, U8 7SEGMENT_CA

Commit message: Finish first prototype version
Parts:
- removed the REF** at (142.9, 88.0)
- removed the REF** at (143.6, 88.0)
- removed the REF** at (140.8, 82.2)
- removed the REF** at (140.8, 83.0)
- removed the REF** at (141.4, 82.0)
- removed the REF** at (142.2, 82.0)
- added REF**: VIA-0.7x0.35, vias:VIA-0.7x0.35, F.Cu at (116.7, 70.1)
- added REF**: VIA-0.7x0.35, vias:VIA-0.7x0.35, F.Cu at (137.7, 90.6)
- added REF**: VIA-0.7x0.35, vias:VIA-0.7x0.35, F.Cu at (138.4, 90.6)
- added REF**: VIA-0.7x0.35, vias:VIA-0.7x0.35, F.Cu at (138.4, 89.9)
- added REF**: VIA-0.7x0.35, vias:VIA-0.7x0.35, F.Cu at (127.2, 91.3)
- added REF**: VIA-0.7x0.35, vias:VIA-0.7x0.35, F.Cu at (128.0, 91.3)
- added REF**: VIA-0.7x0.35, vias:VIA-0.7x0.35, F.Cu at (79.3, 91.0)
- added REF**: VIA-0.7x0.35, vias:VIA-0.7x0.35, F.Cu at (79.3, 88.5)
- added REF**: VIA-0.7x0.35, vias:VIA-0.7x0.35, F.Cu at (79.3, 87.2)
- added REF**: VIA-0.7x0.35, vias:VIA-0.7x0.35, F.Cu at (93.7, 91.3)
- added REF**: VIA-0.7x0.35, vias:VIA-0.7x0.35, F.Cu at (92.9, 91.3)
- added REF**: VIA-0.7x0.35, vias:VIA-0.7x0.35, F.Cu at (106.5, 70.1)
- added REF**: VIA-0.7x0.35, vias:VIA-0.7x0.35, F.Cu at (92.1, 91.3)
- added REF**: VIA-0.7x0.35, vias:VIA-0.7x0.35, F.Cu at (154.3, 87.5)
- added REF**: VIA-0.7x0.35, vias:VIA-0.7x0.35, F.Cu at (140.7, 89.1)
- added REF**: VIA-0.7x0.35, vias:VIA-0.7x0.35, F.Cu at (143.2, 89.6)
- added REF**: VIA-0.7x0.35, vias:VIA-0.7x0.35, F.Cu at (143.9, 88.9)
- added REF**: VIA-0.7x0.35, vias:VIA-0.7x0.35, F.Cu at (143.2, 88.9)
- added REF**: VIA-0.7x0.35, vias:VIA-0.7x0.35, F.Cu at (137.1, 87.5)
- added REF**: VIA-0.7x0.35, vias:VIA-0.7x0.35, F.Cu at (137.1, 86.8)
- added REF**: VIA-0.7x0.35, vias:VIA-0.7x0.35, F.Cu at (94.6, 72.3)
- added REF**: VIA-0.7x0.35, vias:VIA-0.7x0.35, F.Cu at (94.6, 71.5)
- added REF**: VIA-0.7x0.35, vias:VIA-0.7x0.35, F.Cu at (96.3, 70.1)
- added REF**: VIA-0.7x0.35, vias:VIA-0.7x0.35, F.Cu at (95.2, 69.0)
- added REF**: VIA-0.7x0.35, vias:VIA-0.7x0.35, F.Cu at (100.0, 69.0)
- added REF**: VIA-0.7x0.35, vias:VIA-0.7x0.35, F.Cu at (99.3, 69.0)
- added REF**: VIA-0.7x0.35, vias:VIA-0.7x0.35, F.Cu at (115.2, 69.0)
- added REF**: VIA-0.7x0.35, vias:VIA-0.7x0.35, F.Cu at (115.9, 69.0)
- added REF**: VIA-0.7x0.35, vias:VIA-0.7x0.35, F.Cu at (105.0, 69.0)
- added REF**: VIA-0.7x0.35, vias:VIA-0.7x0.35, F.Cu at (105.7, 69.0)
- added REF**: VIA-0.7x0.35, vias:VIA-0.7x0.35, F.Cu at (110.2, 69.0)
- added REF**: VIA-0.7x0.35, vias:VIA-0.7x0.35, F.Cu at (109.5, 69.0)
- added REF**: VIA-0.7x0.35, vias:VIA-0.7x0.35, F.Cu at (120.4, 69.0)
- added REF**: VIA-0.7x0.35, vias:VIA-0.7x0.35, F.Cu at (88.9, 70.1)
- added REF**: VIA-0.7x0.35, vias:VIA-0.7x0.35, F.Cu at (119.7, 69.0)
- added REF**: VIA-0.7x0.35, vias:VIA-0.7x0.35, F.Cu at (91.3, 91.3)
- added REF**: VIA-0.7x0.35, vias:VIA-0.7x0.35, F.Cu at (128.8, 91.3)
- added REF**: VIA-0.7x0.35, vias:VIA-0.7x0.35, F.Cu at (126.4, 91.3)
- added REF**: VIA-0.7x0.35, vias:VIA-0.7x0.35, F.Cu at (137.1, 85.4)
- added REF**: VIA-0.7x0.35, vias:VIA-0.7x0.35, F.Cu at (137.1, 84.7)
- added REF**: VIA-0.7x0.35, vias:VIA-0.7x0.35, F.Cu at (140.1, 83.7)
- added REF**: VIA-0.7x0.35, vias:VIA-0.7x0.35, F.Cu at (142.6, 83.6)
- added REF**: VIA-0.7x0.35, vias:VIA-0.7x0.35, F.Cu at (145.7, 84.2)
- added REF**: VIA-0.7x0.35, vias:VIA-0.7x0.35, F.Cu at (145.7, 84.9)
- added REF**: VIA-0.7x0.35, vias:VIA-0.7x0.35, F.Cu at (88.2, 70.1)
- added REF**: VIA-0.7x0.35, vias:VIA-0.7x0.35, F.Cu at (143.8, 84.2)
- added REF**: VIA-0.7x0.35, vias:VIA-0.7x0.35, F.Cu at (143.8, 84.9)
- added REF**: VIA-0.7x0.35, vias:VIA-0.7x0.35, F.Cu at (140.0, 85.1)
- added REF**: VIA-0.7x0.35, vias:VIA-0.7x0.35, F.Cu at (142.6, 85.7)
- added REF**: VIA-0.7x0.35, vias:VIA-0.7x0.35, F.Cu at (131.7, 78.0)
- added REF**: VIA-0.7x0.35, vias:VIA-0.7x0.35, F.Cu at (88.8, 78.2)
- added REF**: VIA-0.7x0.35, vias:VIA-0.7x0.35, F.Cu at (87.5, 78.8)
- added REF**: VIA-0.7x0.35, vias:VIA-0.7x0.35, F.Cu at (86.6, 83.1)
- added REF**: VIA-0.7x0.35, vias:VIA-0.7x0.35, F.Cu at (86.6, 77.0)
- added REF**: VIA-0.7x0.35, vias:VIA-0.7x0.35, F.Cu at (86.6, 77.7)
- added REF**: VIA-0.7x0.35, vias:VIA-0.7x0.35, F.Cu at (123.0, 70.1)
- added REF**: VIA-0.7x0.35, vias:VIA-0.7x0.35, F.Cu at (70.4, 91.7)
- added REF**: VIA-0.7x0.35, vias:VIA-0.7x0.35, F.Cu at (69.0, 91.7)
- added REF**: VIA-0.7x0.35, vias:VIA-0.7x0.35, F.Cu at (69.7, 91.7)
- added REF**: VIA-0.7x0.35, vias:VIA-0.7x0.35, F.Cu at (66.6, 91.7)
- added REF**: VIA-0.7x0.35, vias:VIA-0.7x0.35, F.Cu at (65.2, 91.7)
- added REF**: VIA-0.7x0.35, vias:VIA-0.7x0.35, F.Cu at (65.9, 91.7)
- added REF**: VIA-0.7x0.35, vias:VIA-0.7x0.35, F.Cu at (65.2, 69.9)
- added REF**: VIA-0.7x0.35, vias:VIA-0.7x0.35, F.Cu at (66.6, 69.9)
- added REF**: VIA-0.7x0.35, vias:VIA-0.7x0.35, F.Cu at (65.9, 69.9)
- added REF**: VIA-0.7x0.35, vias:VIA-0.7x0.35, F.Cu at (69.0, 69.9)
- added REF**: VIA-0.7x0.35, vias:VIA-0.7x0.35, F.Cu at (122.3, 70.1)
- added REF**: VIA-0.7x0.35, vias:VIA-0.7x0.35, F.Cu at (70.4, 69.9)
- added REF**: VIA-0.7x0.35, vias:VIA-0.7x0.35, F.Cu at (69.7, 69.9)
- added REF**: VIA-0.7x0.35, vias:VIA-0.7x0.35, F.Cu at (85.4, 75.4)
- added REF**: VIA-0.7x0.35, vias:VIA-0.7x0.35, F.Cu at (81.6, 75.4)
- added REF**: VIA-0.7x0.35, vias:VIA-0.7x0.35, F.Cu at (86.6, 82.4)
- added REF**: VIA-0.7x0.35, vias:VIA-0.7x0.35, F.Cu at (84.7, 84.2)
- added REF**: VIA-0.7x0.35, vias:VIA-0.7x0.35, F.Cu at (85.3, 83.2)
- added REF**: VIA-0.7x0.35, vias:VIA-0.7x0.35, F.Cu at (83.2, 81.1)
- added REF**: VIA-0.7x0.35, vias:VIA-0.7x0.35, F.Cu at (82.2, 80.1)
- added REF**: VIA-0.7x0.35, vias:VIA-0.7x0.35, F.Cu at (82.2, 82.1)
- added REF**: VIA-0.7x0.35, vias:VIA-0.7x0.35, F.Cu at (133.1, 80.8)
- added REF**: VIA-0.7x0.35, vias:VIA-0.7x0.35, F.Cu at (84.2, 82.1)
- added REF**: VIA-0.7x0.35, vias:VIA-0.7x0.35, F.Cu at (84.2, 80.1)
- added REF**: VIA-0.7x0.35, vias:VIA-0.7x0.35, F.Cu at (81.1, 83.2)
- added REF**: VIA-0.7x0.35, vias:VIA-0.7x0.35, F.Cu at (80.2, 79.6)
- added REF**: VIA-0.7x0.35, vias:VIA-0.7x0.35, F.Cu at (77.3, 79.1)
- added REF**: VIA-0.7x0.35, vias:VIA-0.7x0.35, F.Cu at (77.3, 82.5)
- added REF**: VIA-0.7x0.35, vias:VIA-0.7x0.35, F.Cu at (156.6, 85.6)
- added REF**: VIA-0.7x0.35, vias:VIA-0.7x0.35, F.Cu at (156.6, 84.9)
- added REF**: VIA-0.7x0.35, vias:VIA-0.7x0.35, F.Cu at (156.4, 83.9)
- added REF**: VIA-0.7x0.35, vias:VIA-0.7x0.35, F.Cu at (155.8, 88.9)
- added REF**: VIA-0.7x0.35, vias:VIA-0.7x0.35, F.Cu at (137.7, 89.9)
- added REF**: VIA-0.7x0.35, vias:VIA-0.7x0.35, F.Cu at (155.8, 88.2)
- P3, P4, SW1: footprint terminal:PM_5.08_2 -> Pin_Headers:Pin_Header_Straight_1x02_Pitch2.54mm
- moved P4 193.5 mm to (78.3, 71.1), turned to 270 degrees
- moved R22 188.6 mm to (88.7, 91.0)
- moved C26 134.9 mm to (106.4, 70.1), turned to 180 degrees
- moved RN2 134.8 mm to (131.3, 81.2), turned to 180 degrees
- moved C28 125.1 mm to (116.6, 70.1), turned to 180 degrees
- moved C30 121.3 mm to (96.2, 70.1), turned to 180 degrees
- moved Q10 121.2 mm to (127.6, 86.1)
- moved C29 119.4 mm to (98.6, 69.8), turned to 90 degrees
- moved RN4 116.4 mm to (92.5, 70.8), turned to 180 degrees
- moved Q12 116.3 mm to (92.5, 74.7), turned to 180 degrees
- moved Q3 114.0 mm to (127.6, 74.7)
- moved Q2 111.7 mm to (127.6, 78.5)
- moved RN5 110.3 mm to (127.6, 70.8), turned to 180 degrees
- moved Q11 110.2 mm to (99.9, 70.1), turned to 180 degrees
- moved C25 109.7 mm to (108.8, 69.8), turned to 90 degrees
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Connections:
- L2 pad 1: Net-(D3-Pad2) -> Net-(D4-Pad1)
- L2 pad 2: Net-(D4-Pad1) -> Net-(D3-Pad2)
- L2 pad 3: Net-(D6-Pad1) -> Net-(D5-Pad2)
- L2 pad 4: Net-(D5-Pad2) -> Net-(D6-Pad1)
- Q11 pad 1: /7SEG_2 -> /7SEG_0
- Q4 pad 1: /7SEG_0 -> /7SEG_1
- Q7 pad 1: /7SEG_1 -> /7SEG_2
- RN1 pad 5: /7SEG_D -> /7SEG_E
- RN1 pad 6: /7SEG_C -> /7SEG_D
- RN1 pad 7: /7SEG_B -> /7SEG_C
- RN1 pad 8: /7SEG_A -> /7SEG_DP
- RN2 pad 5: Net-(Q6-Pad3) -> Net-(Q3-Pad3)
- RN2 pad 6: Net-(Q5-Pad3) -> Net-(Q2-Pad3)
- RN2 pad 7: Net-(Q3-Pad3) -> Net-(Q9-Pad3)
- RN2 pad 8: Net-(Q2-Pad3) -> Net-(Q10-Pad3)
- RN3 pad 5: /7SEG_DP -> /7SEG_B
- RN3 pad 6: /7SEG_G -> /7SEG_A
- RN3 pad 8: /7SEG_E -> /7SEG_G
- RN4 pad 5: Net-(Q12-Pad3) -> Net-(Q8-Pad3)
- RN4 pad 6: Net-(Q10-Pad3) -> Net-(Q6-Pad3)
- RN4 pad 7: Net-(Q9-Pad3) -> Net-(Q5-Pad3)
- RN4 pad 8: Net-(Q8-Pad3) -> Net-(Q12-Pad3)
- U4 pad 14: /7SEG_A -> /7SEG_F
- U4 pad 15: /7SEG_B -> /7SEG_G
- U4 pad 26: /7SEG_C -> /7SEG_E
- U4 pad 28: /7SEG_E -> /7SEG_C
- U4 pad 29: /7SEG_F -> /7SEG_DP
- U4 pad 30: /7SEG_G -> /7SEG_A
- U4 pad 31: /7SEG_DP -> /7SEG_B
Routing:
- net GND: track 21.0 -> 118.0 mm
- net /7SEG_DP: track 0.00 -> 76.6 mm, vias 0 -> 2
- net /SYS_SWCLK: track 0.00 -> 73.1 mm, vias 0 -> 2
- net /SPI1_MOSI: track 0.00 -> 72.5 mm, vias 0 -> 2
- net /SYS_SWDIO: track 0.00 -> 71.5 mm, vias 0 -> 2
- net /SPI1_PWR: track 0.00 -> 71.3 mm, vias 0 -> 2
- net /7SEG_C: track 0.00 -> 70.6 mm, vias 0 -> 2
- net /SPI1_SCK: track 0.00 -> 70.0 mm, vias 0 -> 2
- net /SPI1_MISO: track 0.00 -> 69.0 mm, vias 0 -> 2
- net /SPI1_CS: track 0.00 -> 67.9 mm, vias 0 -> 2
- net /SPI1_DR: track 0.00 -> 67.5 mm, vias 0 -> 2
- net /7SEG_D: track 0.00 -> 63.9 mm, vias 0 -> 2
- net /7SEG_E: track 0.00 -> 62.0 mm, vias 0 -> 3
- net /SYS_NRST: track 7.25 -> 66.5 mm, vias 0 -> 2
- net Net-(Q12-Pad1): track 0.00 -> 50.3 mm, vias 0 -> 4
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- added copper zone on B.Cu, net +3V3
- added copper zone on F.Cu, net +3V3
- added copper zone on F.Cu, net +BATT
- added copper zone on B.Cu, net GND
- added copper zone on F.Cu, net Net-(C3-Pad1)
- added copper zone on B.Cu, net Net-(C6-Pad1)
- added copper zone on F.Cu, net Net-(C6-Pad1)
- added copper zone on F.Cu, net Net-(L1-Pad1)
- added copper zone on F.Cu, net Net-(L1-Pad2)
Other:
- board outline added: 102 x 24.4 mm
- net class Default: clearance 0.2 -> 0.15
- rule trace_clearance: 0.2 -> 0.15
- board text added: "None of that Fahrenheit rubbish!"
- board text added: "ROFLtemp-1"
